Commit message: update

File: bobo_description/urdf/robot2_ros2_control.xacro (robot description, xacro)
@@ -4,15 +4,18 @@
     <ros2_control name="${name}" type="system">
         <hardware>
-            <plugin>stm32f1_system_interface/DiffDriveStm32Hardware</plugin>
-            <param name="left_wheel_name">left_wheel_joint</param>
-            <param name="right_wheel_name">right_wheel_joint</param>
+            <plugin>stm32f4_system_interface_gpio/Stm32Hardware</plugin>
+            <param name="left_wheel_name">wheel_left_joint</param>
+            <param name="right_wheel_name">wheel_right_joint</param>
             <param name="loop_rate">40</param>
             <param name="device">/dev/robotController</param>
-            <!--<param name="device">/dev/robotController</param> -->
+            <!--<param name="device">/dev/ROBOTCOM</param> -->
+            <!--<param name="device">/dev/ttyS0</param> -->
+            <!--<param name="device">/dev/ttyUSB0</param> -->
             <param name="baud_rate">115200</param>
             <param name="timeout_ms">1000</param>
             <param name="enc_counts_per_rev">6533</param>
+            <param name="base_width">0.305</param><!-- to edit -->
         </hardware>
-        <joint name="left_wheel_joint">
+        <joint name="wheel_left_joint">
             <command_interface name="velocity">
                 <param name="min">-50</param>
@@ -22,5 +25,5 @@
             <state_interface name="velocity"/>
         </joint>
-        <joint name="right_wheel_joint">
+        <joint name="wheel_right_joint">
             <command_interface name="velocity">
                 <param name="min">-50</param>
