Commit message: update

File: bobo_description/urdf/robot1_ros2_control.xacro (robot description, xacro)
@@ -5,16 +5,16 @@
         <hardware>
             <plugin>stm32f4_system_interface_gpio/Stm32Hardware</plugin>
-            <param name="left_wheel_name">left_wheel_joint</param>
-            <param name="right_wheel_name">right_wheel_joint</param>
+            <param name="left_wheel_name">wheel_left_joint</param>
+            <param name="right_wheel_name">wheel_right_joint</param>
             <param name="loop_rate">40</param>
-            <param name="device">/dev/robotController</param>
-            <!--<param name="device">/dev/ROBOTCOM</param> -->
+            <!-- <param name="device">/dev/robotController</param>  -->
+            <param name="device">/dev/ROBOTCOM</param>
             <!--<param name="device">/dev/ttyS0</param> -->
             <!--<param name="device">/dev/ttyUSB0</param> -->
             <param name="baud_rate">115200</param>
             <param name="timeout_ms">1000</param>
-            <param name="enc_counts_per_rev">6533</param>
+            <param name="enc_counts_per_rev">4096</param>
         </hardware>
-        <joint name="left_wheel_joint">
+        <joint name="wheel_left_joint">
             <command_interface name="velocity">
                 <param name="min">-50</param>
@@ -24,5 +24,5 @@
             <state_interface name="velocity"/>
         </joint>
-        <joint name="right_wheel_joint">
+        <joint name="wheel_right_joint">
             <command_interface name="velocity">
                 <param name="min">-50</param>

File: bobo_description/urdf/robot2_ros2_control.xacro (robot description, xacro)
@@ -8,11 +8,11 @@
             <param name="right_wheel_name">wheel_right_joint</param>
             <param name="loop_rate">40</param>
-            <param name="device">/dev/robotController</param>
-            <!--<param name="device">/dev/ROBOTCOM</param> -->
+            <!-- <param name="device">/dev/robotController</param>  -->
+            <param name="device">/dev/ROBOTCOM</param>
             <!--<param name="device">/dev/ttyS0</param> -->
             <!--<param name="device">/dev/ttyUSB0</param> -->
             <param name="baud_rate">115200</param>
             <param name="timeout_ms">1000</param>
-            <param name="enc_counts_per_rev">6533</param>
+            <param name="enc_counts_per_rev">4096</param>
             <param name="base_width">0.305</param><!-- to edit -->
         </hardware>

Commit message: update

File: bobo_description/urdf/robot1_ros2_control.xacro (robot description, xacro)
@@ -4,5 +4,5 @@
     <ros2_control name="${name}" type="system">
         <hardware>
-            <plugin>stm32f4_system_interface_gpio/Stm32Hardware</plugin>
+            <plugin>bobo_hardware/Stm32Hardware</plugin>
             <param name="left_wheel_name">wheel_left_joint</param>
             <param name="right_wheel_name">wheel_right_joint</param>

File: bobo_description/urdf/robot2.xacro (robot description, xacro)
@@ -51,5 +51,5 @@
   </link>
   <link
-    name="wheel_right_link">
+    name="right_wheel_link">
     <inertial>
       <origin
@@ -91,5 +91,5 @@
   </link>
   <joint
-    name="wheel_right_joint"
+    name="right_wheel_joint"
     type="continuous">
     <origin
@@ -99,10 +99,10 @@
       link="base_link" />
     <child
-      link="wheel_right_link" />
+      link="right_wheel_link" />
     <axis
       xyz="0 -1 0" />
   </joint>
   <link
-    name="wheel_left_link">
+    name="left_wheel_link">
     <inertial>
       <origin
@@ -144,5 +144,5 @@
   </link>
   <joint
-    name="wheel_left_joint"
+    name="left_wheel_joint"
     type="continuous">
     <origin
@@ -152,5 +152,5 @@
       link="base_link" />
     <child
-      link="wheel_left_link" />
+      link="left_wheel_link" />
     <axis
       xyz="0 -1 0" />

File: bobo_description/urdf/robot2_ros2_control.xacro (robot description, xacro)
@@ -1,37 +1,57 @@
 <?xml version="1.0"?>
 <robot xmlns:xacro="http://www.ros.org/wiki/xacro">
-    <xacro:macro name="bobobot_ros2_control" params="name prefix">
+  <xacro:macro name="bobobot_ros2_control" params="name prefix">
     <ros2_control name="${name}" type="system">
-        <hardware>
-            <plugin>stm32f4_system_interface_gpio/Stm32Hardware</plugin>
-            <param name="left_wheel_name">wheel_left_joint</param>
-            <param name="right_wheel_name">wheel_right_joint</param>
-            <param name="loop_rate">40</param>
-            <!-- <param name="device">/dev/robotController</param>  -->
-            <param name="device">/dev/ROBOTCOM</param>
-            <!--<param name="device">/dev/ttyS0</param> -->
-            <!--<param name="device">/dev/ttyUSB0</param> -->
-            <param name="baud_rate">115200</param>
-            <param name="timeout_ms">1000</param>
-            <param name="enc_counts_per_rev">4096</param>
-            <param name="base_width">0.305</param><!-- to edit -->
-        </hardware>
-        <joint name="wheel_left_joint">
-            <command_interface name="velocity">
-                <param name="min">-50</param>
-                <param name="max">50</param>
-            </command_interface>
-            <state_interface name="position"/>
-            <state_interface name="velocity"/>
-        </joint>
-        <joint name="wheel_right_joint">
-            <command_interface name="velocity">
-                <param name="min">-50</param>
-                <param name="max">50</param>
-            </command_interface>
-            <state_interface name="position"/>
-            <state_interface name="velocity"/>
-        </joint>
+      <hardware>
+        <plugin>bobo_hardware/Stm32Hardware</plugin>
+        <param name="left_wheel_name">left_wheel_joint</param>
+        <param name="right_wheel_name">right_wheel_joint</param>
+        <param name="loop_rate">10</param>
+        <param name="device">/dev/ROBOTCOM</param>
+        <!-- <param name="device">/dev/ttyUSB0</param> -->
+        <!-- <param name="device">/dev/ttyACM0</param> -->
+        <param name="baud_rate">115200</param>
+        <param name="timeout_ms">1000</param>
+        <param name="enc_counts_per_rev">4096</param>
+        <param name="pid_p">20</param>
+        <param name="pid_d">12</param>
+        <param name="pid_i">0</param>
+        <param name="pid_o">50</param>
+        <param name="led_max_volt">5</param>
+        <param name="led_min_volt">0</param>
+      </hardware>
+      <joint name="${prefix}left_wheel_joint">
+        <command_interface name="velocity"/>
+        <state_interface name="position"/>
+        <state_interface name="velocity"/>
+      </joint>
+      <joint name="${prefix}right_wheel_joint">
+        <command_interface name="velocity"/>       <!-- diff drive => cm  => stm32f4    -->
+        <state_interface name="position"/>         <!-- stm32f4    => cm  => diff drive -->
+        <state_interface name="velocity"/>
+      </joint>
+      <!-- ROM DYNAMICS ADD -->
+      <gpio name="led1">
+        <command_interface name="digital_command"/>
+        <state_interface   name="digital_status"/>
+      </gpio>
+      <gpio name="led2">
+        <command_interface name="digital_command"/>
+        <state_interface   name="digital_status"/>
+      </gpio>
+      <gpio name="led3">
+        <command_interface name="digital_command"/>
+        <state_interface   name="digital_status"/>
+      </gpio>
+      <gpio name="led4">
+        <command_interface name="digital_command"/>
+        <state_interface   name="digital_status"/>
+      </gpio>
+      <gpio name="estop1">
+        <command_interface name="digital_command"/>
+        <state_interface   name="digital_status"/>
+      </gpio>
+      <!-- ROM DYNAMICS ADD -->
     </ros2_control>
-    </xacro:macro>
+  </xacro:macro>
 </robot>
