Commit message: release-2.0.2-beta

File: bobo_description/urdf/robot1.xacro (robot description, xacro)
@@ -4,5 +4,5 @@
     <link name="base_footprint"/>
     <joint name="base_joint" type="fixed">
-      <origin xyz="0 0 0.0102" rpy="0 0 0" />
+      <origin xyz="0 0 0" rpy="0 0 0" />
       <parent link="base_footprint"/>
       <child link="base_link" />
@@ -31,11 +31,11 @@
       </inertial>
     </link>
-    <joint name="wheel_left_joint" type="continuous">
-      <parent link="base_link"/>
-      <child link="wheel_left_link"/>
+    <joint name="left_wheel_joint" type="continuous">
+      <parent link="base_link"/>
+      <child link="left_wheel_link"/>
       <origin xyz="0.00 ${0.36/2} 0.02" rpy="${-M_PI/2} 0 0"/>
       <axis xyz="0 0 1"/>
     </joint>
-    <link name="wheel_left_link">
+    <link name="left_wheel_link">
       <visual>
         <geometry>
@@ -59,11 +59,11 @@
       </inertial>
     </link>
-    <joint name="wheel_right_joint" type="continuous">
-      <parent link="base_link"/>
-      <child link="wheel_right_link"/>
+    <joint name="right_wheel_joint" type="continuous">
+      <parent link="base_link"/>
+      <child link="right_wheel_link"/>
       <origin xyz="0.00 -${0.36/2} 0.02" rpy="${-M_PI/2} 0 0"/>
       <axis xyz="0 0 1"/>
     </joint>
-    <link name="wheel_right_link">
+    <link name="right_wheel_link">
       <visual>
         <geometry>
@@ -141,10 +141,40 @@
       </inertial>
     </link>
-    <joint name="imu_joint" type="fixed">
+    <!-- ROM Edit -->
+    <!-- LASER -->
+    <joint name="laser_joint" type="fixed">
+      <parent link="base_link"/>
+      <child link="laser_link"/>
+      <origin xyz="0.18 0 0.24" rpy="3.1415926 0 0"/>
+    </joint>
+    <link name="laser_link">
+      <visual>
+        <origin xyz="0 0 0.0" rpy="0 0 0"/>
+        <geometry>
+          <box size="0.05 0.05 0.05"/>
+        </geometry>
+        <material name="grey_blue"/>
+      </visual>
+      <collision>
+        <origin xyz="0.015 0 -0.0065" rpy="0 0 0"/>
+        <geometry>
+          <cylinder length="0.0315" radius="0.055"/>
+        </geometry>
+      </collision>
+      <inertial>
+        <mass value="0.114" />
+        <origin xyz="0 0 0" />
+        <inertia ixx="0.001" ixy="0.0" ixz="0.0"
+                 iyy="0.001" iyz="0.0"
+                 izz="0.001" />
+      </inertial>
+    </link>
+  <!-- IMU -->
+  <joint name="imu_joint" type="fixed">
       <parent link="base_link"/>
       <child link="imu_link"/>
       <origin xyz="0 0 0.268" rpy="0 0 0"/>
-    </joint>
-    <link name="imu_link">
+  </joint>
+  <link name="imu_link">
       <visual>
         <origin xyz="0 0 0.0" rpy="0 0 0"/>
@@ -154,32 +184,51 @@
         <material name="red"/>
       </visual>
-    </link>
-    <joint name="laser_joint" type="fixed">
-      <parent link="base_link"/>
-      <child link="laser_link"/>
-      <origin xyz="0.18 0 0.24" rpy="3.1415926 0 0"/>
-    </joint>
-    <link name="laser_link">
-      <visual>
-        <origin xyz="0 0 0.0" rpy="0 0 0"/>
-        <geometry>
-          <box size="0.05 0.05 0.05"/>
-        </geometry>
-        <material name="grey_blue"/>
-      </visual>
-      <collision>
-        <origin xyz="0.015 0 -0.0065" rpy="0 0 0"/>
-        <geometry>
-          <cylinder length="0.0315" radius="0.055"/>
-        </geometry>
-      </collision>
-      <inertial>
-        <mass value="0.114" />
-        <origin xyz="0 0 0" />
-        <inertia ixx="0.001" ixy="0.0" ixz="0.0"
-                 iyy="0.001" iyz="0.0"
-                 izz="0.001" />
-      </inertial>
-    </link>
+  </link>
+  <!-- 3D CAM1 -->
+  <joint name="right_camera_joint" type="fixed">
+    <parent link="base_link"/>
+    <child link="right_camera_link"/>
+    <origint xyz="0.18 -0.2 0.1" rpy="0 0 0"/>
+  </joint>
+  <link name="right_camera_link">
+      <visual>
+        <origin xyz="0 0 0.0" rpy="0 0 0"/>
+        <geometry>
+          <box size="0.03 0.02 0.02"/>
+        </geometry>
+        <material name="blue"/>
+      </visual>
+  </link>
+  <!-- 3D CAM2 -->
+  <joint name="left_camera_joint" type="fixed">
+    <parent link="base_link"/>
+    <child link="left_camera_link"/>
+    <origint xyz="0.18 0.2 0.1" rpy="0 0 0"/>
+  </joint>
+  <link name="left_camera_link">
+      <visual>
+        <origin xyz="0 0 0.0" rpy="0 0 0"/>
+        <geometry>
+          <box size="0.03 0.02 0.02"/>
+        </geometry>
+        <material name="blue"/>
+      </visual>
+  </link>
+  <!-- 3D CAM3 -->
+  <joint name="top_camera_joint" type="fixed">
+    <parent link="base_link"/>
+    <child link="top_camera_link"/>
+    <origint xyz="0.18 0 0.5" rpy="0 0 0"/>
+  </joint>
+  <link name="top_camera_link">
+      <visual>
+        <origin xyz="0 0 0.0" rpy="0 0 0"/>
+        <geometry>
+          <box size="0.03 0.02 0.02"/>
+        </geometry>
+        <material name="blue"/>
+      </visual>
+  </link>
+  <!-- materials colors for rviz  -->
   <material name="white">
     <color rgba="1 1 1 0.8"/>
@@ -212,3 +261,4 @@
     <color rgba="1.0 0.7 0.0 1"/>
   </material>
+  <!-- ROM END -->
 </robot>

File: bobo_description/urdf/robot1_complete.urdf.xacro (robot description, xacro)
@@ -3,7 +3,5 @@
     <xacro:arg name="prefix" default="" />
     <xacro:include filename="$(find bobo_description)/urdf/$(env BOBO_MODEL).xacro" />
-    <!-- <xacro:include filename="robot1.xacro" /> -->
     <xacro:include filename="$(env BOBO_MODEL)_ros2_control.xacro" />
-    <!-- <xacro:include filename="robot1_ros2_control.xacro" /> -->
-    <xacro:bobobot_ros2_control name="bobobot" prefix="$(arg prefix)" />
+    <xacro:diffbot_ros2_control name="DiffBot" prefix="$(arg prefix)" />
 </robot>

File: bobo_description/urdf/robot1_ros2_control.xacro (robot description, xacro)
@@ -1,36 +1,64 @@
 <?xml version="1.0"?>
 <robot xmlns:xacro="http://www.ros.org/wiki/xacro">
-    <xacro:macro name="bobobot_ros2_control" params="name prefix">
+  <xacro:macro name="diffbot_ros2_control" params="name prefix">
     <ros2_control name="${name}" type="system">
-        <hardware>
-            <plugin>bobo_hardware/Stm32Hardware</plugin>
-            <param name="left_wheel_name">wheel_left_joint</param>
-            <param name="right_wheel_name">wheel_right_joint</param>
-            <param name="loop_rate">40</param>
-            <!-- <param name="device">/dev/robotController</param>  -->
-            <param name="device">/dev/ROBOTCOM</param>
-            <!--<param name="device">/dev/ttyS0</param> -->
-            <!--<param name="device">/dev/ttyUSB0</param> -->
-            <param name="baud_rate">115200</param>
-            <param name="timeout_ms">1000</param>
-            <param name="enc_counts_per_rev">4096</param>
-        </hardware>
-        <joint name="wheel_left_joint">
-            <command_interface name="velocity">
-                <param name="min">-50</param>
-                <param name="max">50</param>
-            </command_interface>
-            <state_interface name="position"/>
-            <state_interface name="velocity"/>
-        </joint>
-        <joint name="wheel_right_joint">
-            <command_interface name="velocity">
-                <param name="min">-50</param>
-                <param name="max">50</param>
-            </command_interface>
-            <state_interface name="position"/>
-            <state_interface name="velocity"/>
-        </joint>
+      <hardware>
+        <plugin>bobo_hardware/Stm32Hardware</plugin>
+        <param name="left_wheel_name">left_wheel_joint</param>
+        <param name="right_wheel_name">right_wheel_joint</param>
+        <param name="loop_rate">10</param>
+        <param name="device">/dev/ROBOTCOM</param>
+        <!-- <param name="device">/dev/ttyUSB0</param> -->
+        <!-- <param name="device">/dev/ttyACM0</param> -->
+        <param name="baud_rate">115200</param>
+        <param name="timeout_ms">1000</param>
+        <param name="enc_counts_per_rev">4096</param>
+        <param name="pid_p">0</param>
+        <param name="pid_i">0</param>
+        <param name="pid_d">0</param>
+        <param name="pid_o">0</param>
+        <param name="imu_coef_m_for_positive_degree">0.00550</param>
+        <param name="imu_bias_b_for_positive_degree">-0.2891</param>
+        <param name="imu_coef_m_for_negative_degree">0.00550</param>
+        <param name="imu_bias_b_for_negative_degree">-360.0</param>
+        <param name="imu_period">5.0</param>
+      </hardware>
+      <joint name="${prefix}left_wheel_joint">
+        <command_interface name="velocity"/>
+        <state_interface name="position"/>
+        <state_interface name="velocity"/>
+      </joint>
+      <joint name="${prefix}right_wheel_joint">
+        <command_interface name="velocity"/>       <!-- diff drive => cm  => stm32f4    -->
+        <state_interface name="position"/>         <!-- stm32f4    => cm  => diff drive -->
+        <state_interface name="velocity"/>
+      </joint>
+      <!-- ROM DYNAMICS ADD -->
+      <gpio name="led1">
+        <command_interface name="digital_command"/>
+        <state_interface   name="digital_status"/>
+      </gpio>
+      <gpio name="led2">
+        <command_interface name="digital_command"/>
+        <state_interface   name="digital_status"/>
+      </gpio>
+      <gpio name="led3">
+        <command_interface name="digital_command"/>
+        <state_interface   name="digital_status"/>
+      </gpio>
+      <gpio name="led4">
+        <command_interface name="digital_command"/>
+        <state_interface   name="digital_status"/>
+      </gpio>
+      <gpio name="estop1">
+        <command_interface name="digital_command"/>
+        <state_interface   name="digital_status"/>
+      </gpio>
+      <gpio name="imu1">
+        <command_interface name="digital_command"/>
+        <state_interface   name="digital_status"/>
+      </gpio>
+      <!-- ROM DYNAMICS ADD -->
     </ros2_control>
-    </xacro:macro>
+  </xacro:macro>
 </robot>

File: bobo_description/urdf/robot2_ros2_control.xacro (robot description, xacro)
@@ -1,5 +1,5 @@
 <?xml version="1.0"?>
 <robot xmlns:xacro="http://www.ros.org/wiki/xacro">
-  <xacro:macro name="bobobot_ros2_control" params="name prefix">
+  <xacro:macro name="diffbot_ros2_control" params="name prefix">
     <ros2_control name="${name}" type="system">
       <hardware>
@@ -14,8 +14,8 @@
         <param name="timeout_ms">1000</param>
         <param name="enc_counts_per_rev">4096</param>
-        <param name="pid_p">20</param>
-        <param name="pid_d">12</param>
+        <param name="pid_p">0</param>
         <param name="pid_i">0</param>
-        <param name="pid_o">50</param>
+        <param name="pid_d">0</param>
+        <param name="pid_o">0</param>
         <param name="imu_coef_m_for_positive_degree">0.00550</param>
         <param name="imu_bias_b_for_positive_degree">-0.2891</param>
@@ -23,5 +23,4 @@
         <param name="imu_bias_b_for_negative_degree">-360.0</param>
         <param name="imu_period">5.0</param>
-        <param name="imu_link_name">imu_link</param>
       </hardware>
       <joint name="${prefix}left_wheel_joint">
@@ -56,8 +55,8 @@
         <state_interface   name="digital_status"/>
       </gpio>
-      <!-- IMU -->
-      <sensor name="imu">
-        <state_interface name="yaw_heading"/>
-      </sensor>
+      <gpio name="imu1">
+        <command_interface name="digital_command"/>
+        <state_interface   name="digital_status"/>
+      </gpio>
       <!-- ROM DYNAMICS ADD -->
     </ros2_control>
